Commit message: Updated 2d nav and launch for hydro.\n\nThis uses the chest calibration from strands to put the chest xtion at the right height and angle. There are some odd problems still, notably the laser tf frame jumps about but laserbase is stable, so currently publishing to that instead.

File: bham_b21_launch/b21.urdf (robot description, URDF)
Before this commit: robot lewis, 20 links, 19 joints
Links:
- added link chest_xtion_depth_frame
- added link chest_xtion_depth_optical_frame
- added link chest_xtion_height_tilt_link
- added link chest_xtion_link; collision box size=0.001 0.001 0.001; visual mesh filename=package://scitos_description/meshes/xtion.dae
- added link chest_xtion_rgb_frame
- added link chest_xtion_rgb_optical_frame
Joints:
- added joint chest_xtion_base_link: type fixed, parent chest_xtion_link, child chest_xtion_depth_frame, origin xyz=0 0.045 0 rpy=0 0 0
- added joint chest_xtion_base_link1: type fixed, parent chest_xtion_link, child chest_xtion_rgb_frame, origin xyz=0 0.02 0 rpy=0 0 0
- added joint chest_xtion_base_link2: type fixed, parent chest_xtion_depth_frame, child chest_xtion_depth_optical_frame, origin xyz=0 0 0 rpy=-1.5707963267948966 0 -1.5707963267948966
- added joint chest_xtion_base_link3: type fixed, parent chest_xtion_rgb_frame, child chest_xtion_rgb_optical_frame, origin xyz=0 0 0 rpy=-1.5707963267948966 0 -1.5707963267948966
- added joint chest_xtion_height_joint: type prismatic, parent base_link, child chest_xtion_height_tilt_link, origin xyz=0.43 0 0 rpy=0 0 0, axis 0 0 1, limit lower=0.5 upper=1.5 effort=1000 velocity=1000
- added joint chest_xtion_tilt_joint: type continuous, parent chest_xtion_height_tilt_link, child chest_xtion_link, origin xyz=0 0 0 rpy=0 0 0, axis 0 1 0

File: bham_b21_launch/b21.xacro (robot description, xacro)
@@ -200,3 +200,63 @@
 <xacro:eye prefix="left" sign="" />
 <xacro:eye prefix="right" sign="-" />
+  <!-- Connect base to chest_xtion_link -->
+  <link name="chest_xtion_link">
+    <visual>
+      <origin rpy="3.14 0 0" xyz="0 0 0"/>
+      <geometry>
+        <mesh filename="package://scitos_description/meshes/xtion.dae"/>
+      </geometry>
+    </visual>
+    <collision>
+      <origin rpy="0 0 0" xyz="0 0 0.071"/>
+      <geometry>
+        <box size="0.001 0.001 0.001"/>
+      </geometry>
+    </collision>
+  </link>
+  <link name="chest_xtion_height_tilt_link"/>
+  <joint name="chest_xtion_height_joint" type="prismatic" >
+    <!-- Z height from calibrate_chest -->
+    <axis xyz="0 0 1"/>
+    <origin rpy="0 0 0" xyz="0.43 0 0" />
+    <limit effort="1000" velocity="1000" lower="0.5" upper="1.5"/>
+    <parent link="base_link"/>
+    <child link="chest_xtion_height_tilt_link"/>
+  </joint>
+  <joint name="chest_xtion_tilt_joint" type="continuous" >
+    <!-- Rotation y angle from calibrate_chest-->
+    <axis xyz="0 1 0"/>
+    <origin rpy="0 0 0" xyz="0 0 0" />
+    <parent link="chest_xtion_height_tilt_link"/>
+    <child link="chest_xtion_link"/>
+  </joint>
+  <!-- chest_xtion internal frames -->
+  <link name="chest_xtion_depth_frame"/>
+  <link name="chest_xtion_rgb_frame"/>
+  <link name="chest_xtion_depth_optical_frame"/>
+  <link name="chest_xtion_rgb_optical_frame"/>
+  <joint name="chest_xtion_base_link" type="fixed" >
+    <origin rpy="0 0 0"
+            xyz="0 0.045 0" />
+    <parent link="chest_xtion_link"/>
+    <child link="chest_xtion_depth_frame"/>
+  </joint>
+  <joint name="chest_xtion_base_link1" type="fixed" >
+    <origin rpy="0 0 0"
+            xyz="0 0.02 0" />
+    <parent link="chest_xtion_link"/>
+    <child link="chest_xtion_rgb_frame"/>
+  </joint>
+  <joint name="chest_xtion_base_link2" type="fixed" >
+    <origin rpy="-1.5707963267948966 0 -1.5707963267948966"
+            xyz="0 0 0" />
+    <parent link="chest_xtion_depth_frame"/>
+    <child link="chest_xtion_depth_optical_frame"/>
+  </joint>
+  <joint name="chest_xtion_base_link3" type="fixed" >
+    <origin rpy="-1.5707963267948966 0 -1.5707963267948966"
+            xyz="0 0 0" />
+    <parent link="chest_xtion_rgb_frame"/>
+    <child link="chest_xtion_rgb_optical_frame"/>
+  </joint>
 </robot>
